File: kicad/asynthosc/ethernet.kicad_sch (KiCad schematic)
At the start: 4 parts, among them J3 RJ45_LED, U5 LAN8742A, U6 USBLC6-2P6

Commit message: sch: rmii side
Parts:
- added C31, C32: 30pF, 0402, symbol Device:C
- added C33: 470pF, 0402, symbol Device:C
- added C34: 1uF, 0402, symbol Device:C
- added C35, C36, C37, C39, C40, C41: 100nF, 0402, symbol Device:C
- added C42: 1000pF X7R, 1206, symbol Device:C
- added C43: 10uF, symbol Device:C_Polarized
- added FB3: BLM15PX330SN1D, 0402, symbol Device:FerriteBead
- added JP4: SolderJumper_2_Bridged, symbol Jumper:SolderJumper_2_Bridged
- added R35, R36, R37, R38, R45: 33R, 0402, symbol Device:R
- added R46, R47, R49: 100k, 0402, symbol Device:R
- added R48: 1.5K, 0402, symbol Device:R
- added R50: 12.1k, 0402, symbol Device:R
- added R51, R52, R53, R54: 75R, 0402, symbol Device:R
- added R55, R56: 270R, 0402, symbol Device:R
- added R57, R58, R59, R60: 50R, 0402, symbol Device:R
- added Y2: 25MHZ,20PF,30PPM, symbol Device:Crystal
Connections:
- net RX_P: now reaches U6.1 (I/O1)
- net RX_P: now also TR1.3 (TD-), U5.23 (RXP), R58.1
- net GND: now reaches U6.2 (GND)
- net GND: now also U5.25 (VSS), C31.1, C32.1, C33.2, C34.2, C35.2, C36.2, C37.2, C39.2, C40.2, C41.2, C42.2, C43.2, R37.1, R50.2, R55.1, R56.1
- net TX_P: now reaches U6.3 (I/O2)
- net TX_P: now also TR1.8 (RD-), U5.21 (TXP), R60.1
- net TX_N: now reaches U6.4 (I/O2)
- net TX_N: now also TR1.6 (RD+), U5.20 (TXN), R59.1
- net 3V3_FILT: now reaches U6.5 (VBUS)
- net 3V3_FILT: now also TR1.2 (C_TD), TR1.7 (C_RD), U5.1 (VDD2A), U5.19 (VDD1A), C36.1, C37.1, C39.1, C40.1, C41.1, C43.1, FB3.1, R57.2, R58.2, R59.2, R60.2
- net RX_N: now reaches U6.6 (I/O1)
- net RX_N: now also TR1.1 (TD+), U5.22 (RXN), R57.1
- net RJ_TX_P: now reaches J3.1
- net RJ_TX_P: now also TR1.9 (RX-)
- net RJ45_LED2: now reaches J3.10
- net RJ45_LED2: now also U5.2 (LED2/~{INTSEL})
- net at J3.11: now also R56.2
- net RJ45_LED1: now reaches J3.12
- net RJ45_LED1: now also U5.3 (LED1/REGOFF)
- net RJ_TX_N: now reaches J3.2
- net RJ_TX_N: now also TR1.11 (RX+)
- net RJ_RX_P: now reaches J3.3
- net RJ_RX_P: now also TR1.14 (TX-)
- net at J3.4: now also J3.5, R53.2
- net RJ_RX_N: now reaches J3.6
- net RJ_RX_N: now also TR1.15 (C_TX), R51.2
- net at J3.7: now also J3.8, R54.2
- net at J3.9: now also R55.2
- net at TR1.10 (C_RX): now also R52.2
- net at U5.10 (RXER/PHYAD0): now also R37.2
- net at U5.11 (CRS_DV/MODE2): now also R38.2
- net RMII_MDIO: now reaches U5.12 (MDIO)
- net RMII_MDIO: now also R48.1
- net RMII_MDC: now reaches U5.13 (MDC)
- net at U5.14 (~{INT}/REFCLKO): now also R45.2
- net at U5.15 (~{RST}): now also JP4.1 (A)
- net RMII_TX_EN: now reaches U5.16 (TXEN)
- net RMII_TXD0: now reaches U5.17 (TXD0)
- net RMII_TXD1: now reaches U5.18 (TXD1)
- net at U5.24 (RBIAS): now also R50.1
- net at U5.4 (XTAL2): now also C32.2, Y2.2
- net at U5.5 (XTAL1/CLKIN): now also C31.2, Y2.1
- net 3V3: now reaches U5.6 (VDDCR)
- net 3V3: now also U5.9 (VDDIO), C33.1, C34.1, C35.1, FB3.2, R46.2, R47.2, R48.2, R49.2
- net at U5.7 (RXD1/MODE1): now also R36.2
- net at U5.8 (RXD0/MODE0): now also R35.2
- new net: C42.1, R51.1, R52.1, R53.1, R54.1
- new net RMII_CRS_DV: R38.1
- new net RMII_NRST: JP4.2 (B)
- new net RMII_REF_CLK: R45.1, R49.1
- new net RMII_RXD0: R35.1, R46.1
- new net RMII_RXD1: R36.1, R47.1
Other:
- note added: "bead,600R,350mA,0603,FCM1608KF-601T05"
- moved on the sheet: J3, TR1, U5, U6

Commit message: sch: update and new interface sheet
Parts:
- C31, C32, C33, C34, C35, C36, C37, C39, C40, C41, FB3, R35, R36, R37, R38, R45, R46, R47, R48, R49, R50, R51, R52, R53, R54, R55, R56, R57, R58, R59, R60: footprint 0402 -> (none)
- C42: footprint 1206 -> (none)
Changed lines of the file:
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@@
 			)
 		)
-		(property "Footprint" "0402"
+		(property "Footprint" ""
 			(at 107.6452 147.32 0)
 			(effects
@@
 			)
 		)
-		(property "Footprint" "0402"
+		(property "Footprint" ""
 			(at 37.338 54.61 90)
 			(effects
@@
 			)
 		)
-		(property "Footprint" "0402"
+		(property "Footprint" ""
 			(at 57.15 84.328 90)
 			(effects
@@
 			)
 		)
-		(property "Footprint" "0402"
+		(property "Footprint" ""
 			(at 57.15 81.788 90)
 			(effects
@@
 			)
 		)
-		(property "Footprint" "0402"
+		(property "Footprint" ""
 			(at 100.0252 147.32 0)
 			(effects
@@
 			)
 		)
-		(property "Footprint" "0402"
+		(property "Footprint" ""
 			(at 57.15 76.708 90)
 			(effects
@@
 			)
 		)
-		(property "Footprint" "0402"
+		(property "Footprint" ""
 			(at 57.15 79.248 90)
 			(effects
@@
 			)
 		)
-		(property "Footprint" "0402"
+		(property "Footprint" ""
 			(at 189.738 91.44 90)
 			(effects
@@
 			)
 		)
-		(property "Footprint" "0402"
+		(property "Footprint" ""
 			(at 54.9148 120.65 0)
 			(effects
@@
 			)
 		)
-		(property "Footprint" "0402"
+		(property "Footprint" ""
 			(at 117.348 59.69 90)
 			(effects
@@
 			)
 		)
-		(property "Footprint" "0402"
+		(property "Footprint" ""
 			(at 62.5348 120.65 0)
 			(effects
@@
 			)
 		)
-		(property "Footprint" "0402"
+		(property "Footprint" ""
 			(at 243.078 83.82 90)
 			(effects
@@
 			)
 		)
-		(property "Footprint" "0402"
+		(property "Footprint" ""
 			(at 126.6952 147.32 0)
 			(effects
@@
 			)
 		)
-		(property "Footprint" "1206"
+		(property "Footprint" ""
 			(at 200.3552 111.76 0)
 			(effects
@@
 			)
 		)
-		(property "Footprint" "0402"
+		(property "Footprint" ""
 			(at 122.428 59.69 90)
 			(effects
@@
 			)
 		)
-		(property "Footprint" "0402"
+		(property "Footprint" ""
 			(at 116.84 86.868 90)
 			(effects
@@
 			)
 		)
-		(property "Footprint" "0402"
+		(property "Footprint" ""
 			(at 119.888 59.69 90)
 			(effects
@@
 			)
 		)
-		(property "Footprint" "0402"
+		(property "Footprint" ""
 			(at 152.0952 147.32 0)
 			(effects
@@
 			)
 		)
-		(property "Footprint" "0402"
+		(property "Footprint" ""
 			(at 115.2652 147.32 0)
 			(effects
@@
 		(at 59.69 111.76 0)
 		(unit 1)
-		(exclude_from_sim no)
+		(exclude_from_sim yes)
 		(in_bom yes)
 		(on_board yes)
@@
 			)
 		)
-		(property "Footprint" "0402"
+		(property "Footprint" ""
 			(at 124.968 59.69 90)
 			(effects
@@
 			)
 		)
-		(property "Footprint" "0402"
+		(property "Footprint" ""
 			(at 255.778 83.82 90)
 			(effects
@@
 			)
 		)
-		(property "Footprint" "0402"
+		(property "Footprint" ""
 			(at 193.548 91.44 90)
 			(effects
@@
 			)
 		)
-		(property "Footprint" "0402"
+		(property "Footprint" ""
 			(at 42.418 54.61 90)
 			(effects
@@
 			)
 		)
-		(property "Footprint" "0402"
+		(property "Footprint" ""
 			(at 39.878 54.61 90)
 			(effects
@@
 			)
 		)
-		(property "Footprint" "0402"
+		(property "Footprint" ""
 			(at 210.058 91.44 90)
 			(effects
@@
 			)
 		)
-		(property "Footprint" "0402"
+		(property "Footprint" ""
 			(at 134.3152 147.32 0)
 			(effects
@@
 			)
 		)
-		(property "Footprint" "0402"
+		(property "Footprint" ""
 			(at 158.4452 147.32 0)
 			(effects
@@
 			)
 		)
-		(property "Footprint" "0402"
+		(property "Footprint" ""
 			(at 57.15 97.028 90)
 			(effects
@@
 			)
 		)
-		(property "Footprint" "0402"
+		(property "Footprint" ""
 			(at 213.868 91.44 90)
 			(effects
@@
 			)
 		)
-		(property "Footprint" "0402"
+		(property "Footprint" ""
 			(at 47.498 54.61 90)
 			(effects
@@
 			)
 		)
-		(property "Footprint" "0402"
+		(property "Footprint" ""
 			(at 91.44 29.972 90)
 			(effects
@@
 			)
 		)
-		(property "Footprint" "0402"
+		(property "Footprint" ""
 			(at 201.6252 36.83 0)
 			(effects

Commit message: sch: update footprint links
Parts:
- C31, C32, C33, C35, C36, C37, C39, C40, C41, C42: footprint (none) -> Capacitor_SMD:C_0402_1005Metric
- C34: footprint (none) -> Capacitor_SMD:C_0805_2012Metric
- C43: footprint (none) -> Capacitor_SMD:CP_Elec_4x5.4
- JP4: footprint (none) -> Jumper:SolderJumper-2_P1.3mm_Bridged2Bar_Pad1.0x1.5mm
- R35, R36, R37, R38, R45, R46, R47, R48, R49, R50, R51, R52, R53, R54, R55, R56, R57, R58, R59, R60: footprint (none) -> Resistor_SMD:R_0402_1005Metric
- Y2: footprint (none) -> Crystal:Crystal_SMD_3225-4Pin_3.2x2.5mm
Changed lines of the file:
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@@
 			)
 		)
-		(property "Footprint" ""
+		(property "Footprint" "Capacitor_SMD:C_0805_2012Metric"
 			(at 107.6452 147.32 0)
 			(effects
@@
 			)
 		)
-		(property "Footprint" ""
+		(property "Footprint" "Resistor_SMD:R_0402_1005Metric"
 			(at 37.338 54.61 90)
 			(effects
@@
 			)
 		)
-		(property "Footprint" ""
+		(property "Footprint" "Resistor_SMD:R_0402_1005Metric"
 			(at 57.15 84.328 90)
 			(effects
@@
 			)
 		)
-		(property "Footprint" ""
+		(property "Footprint" "Resistor_SMD:R_0402_1005Metric"
 			(at 57.15 81.788 90)
 			(effects
@@
 			)
 		)
-		(property "Footprint" ""
+		(property "Footprint" "Capacitor_SMD:C_0402_1005Metric"
 			(at 100.0252 147.32 0)
 			(effects
@@
 			)
 		)
-		(property "Footprint" ""
+		(property "Footprint" "Resistor_SMD:R_0402_1005Metric"
 			(at 57.15 76.708 90)
 			(effects
@@
 			)
 		)
-		(property "Footprint" ""
+		(property "Footprint" "Resistor_SMD:R_0402_1005Metric"
 			(at 57.15 79.248 90)
 			(effects
@@
 			)
 		)
-		(property "Footprint" ""
+		(property "Footprint" "Resistor_SMD:R_0402_1005Metric"
 			(at 189.738 91.44 90)
 			(effects
@@
 			)
 		)
-		(property "Footprint" ""
+		(property "Footprint" "Capacitor_SMD:C_0402_1005Metric"
 			(at 54.9148 120.65 0)
 			(effects
@@
 			)
 		)
-		(property "Footprint" ""
+		(property "Footprint" "Resistor_SMD:R_0402_1005Metric"
 			(at 117.348 59.69 90)
 			(effects
@@
 			)
 		)
-		(property "Footprint" ""
+		(property "Footprint" "Capacitor_SMD:C_0402_1005Metric"
 			(at 62.5348 120.65 0)
 			(effects
@@
 			)
 		)
-		(property "Footprint" ""
+		(property "Footprint" "Resistor_SMD:R_0402_1005Metric"
 			(at 243.078 83.82 90)
 			(effects
@@
 			)
 		)
-		(property "Footprint" ""
+		(property "Footprint" "Capacitor_SMD:CP_Elec_4x5.4"
 			(at 141.9352 147.32 0)
 			(effects
@@
 			)
 		)
-		(property "Footprint" ""
+		(property "Footprint" "Capacitor_SMD:C_0402_1005Metric"
 			(at 126.6952 147.32 0)
 			(effects
@@
 			)
 		)
-		(property "Footprint" ""
+		(property "Footprint" "Capacitor_SMD:C_0402_1005Metric"
 			(at 200.3552 111.76 0)
 			(effects
@@
 			)
 		)
-		(property "Footprint" ""
+		(property "Footprint" "Resistor_SMD:R_0402_1005Metric"
 			(at 122.428 59.69 90)
 			(effects
@@
 			)
 		)
-		(property "Footprint" ""
+		(property "Footprint" "Resistor_SMD:R_0402_1005Metric"
 			(at 116.84 86.868 90)
 			(effects
@@
 			)
 		)
-		(property "Footprint" ""
+		(property "Footprint" "Jumper:SolderJumper-2_P1.3mm_Bridged2Bar_Pad1.0x1.5mm"
 			(at 57.15 92.71 0)
 			(effects
@@
 			)
 		)
-		(property "Footprint" ""
+		(property "Footprint" "Resistor_SMD:R_0402_1005Metric"
 			(at 119.888 59.69 90)
 			(effects
@@
 			)
 		)
-		(property "Footprint" ""
+		(property "Footprint" "Capacitor_SMD:C_0402_1005Metric"
 			(at 152.0952 147.32 0)
 			(effects
@@
 			)
 		)
-		(property "Footprint" ""
+		(property "Footprint" "Capacitor_SMD:C_0402_1005Metric"
 			(at 115.2652 147.32 0)
 			(effects
@@
 			)
 		)
-		(property "Footprint" ""
+		(property "Footprint" "Crystal:Crystal_SMD_3225-4Pin_3.2x2.5mm"
 			(at 59.69 111.76 0)
 			(effects
@@
 			)
 		)
-		(property "Footprint" ""
+		(property "Footprint" "Resistor_SMD:R_0402_1005Metric"
 			(at 124.968 59.69 90)
 			(effects
@@
 			)
 		)
-		(property "Footprint" ""
+		(property "Footprint" "Resistor_SMD:R_0402_1005Metric"
 			(at 255.778 83.82 90)
 			(effects
@@
 			)
 		)
-		(property "Footprint" ""
+		(property "Footprint" "Resistor_SMD:R_0402_1005Metric"
 			(at 193.548 91.44 90)
 			(effects
@@
 			)
 		)
-		(property "Footprint" ""
+		(property "Footprint" "Resistor_SMD:R_0402_1005Metric"
 			(at 42.418 54.61 90)
 			(effects
@@
 			)
 		)
-		(property "Footprint" ""
+		(property "Footprint" "Resistor_SMD:R_0402_1005Metric"
 			(at 39.878 54.61 90)
 			(effects
@@
 			)
 		)
-		(property "Footprint" ""
+		(property "Footprint" "Resistor_SMD:R_0402_1005Metric"
 			(at 210.058 91.44 90)
 			(effects
@@
 			)
 		)
-		(property "Footprint" ""
+		(property "Footprint" "Capacitor_SMD:C_0402_1005Metric"
 			(at 134.3152 147.32 0)
 			(effects
@@
 			)
 		)
-		(property "Footprint" ""
+		(property "Footprint" "Capacitor_SMD:C_0402_1005Metric"
 			(at 158.4452 147.32 0)
 			(effects
@@
 			)
 		)
-		(property "Footprint" ""
+		(property "Footprint" "Resistor_SMD:R_0402_1005Metric"
 			(at 57.15 97.028 90)
 			(effects
@@
 			)
 		)
-		(property "Footprint" ""
+		(property "Footprint" "Resistor_SMD:R_0402_1005Metric"
 			(at 213.868 91.44 90)
 			(effects
@@
 			)
 		)
-		(property "Footprint" ""
+		(property "Footprint" "Resistor_SMD:R_0402_1005Metric"
 			(at 47.498 54.61 90)
 			(effects
@@
 			)
 		)
-		(property "Footprint" ""
+		(property "Footprint" "Capacitor_SMD:C_0402_1005Metric"
 			(at 201.6252 36.83 0)
 			(effects

Commit message: wip
Parts:
- removed J3: RJ45_LED, symbol Connector:RJ45_LED
- added J3: RJ45_LED_Shielded, asynthosc:RJ45_HCTL_HC-RJ45-053-2, symbol Connector:RJ45_LED_Shielded
- FB3: footprint (none) -> Inductor_SMD:L_0402_1005Metric
Connections:
- net GND: now also J3.SH
- net RJ45_LED1: now also J3.12
- net RJ45_LED2: now also J3.10
- net RJ_RX_N: now also J3.6
- net RJ_RX_P: now also J3.3
- net RJ_TX_N: now also J3.2
- net RJ_TX_P: now also J3.1
- net at R55.2: now also J3.9
- net at R56.2: now also J3.11
- net at R53.2: now also J3.4, J3.5
- net at R54.2: now also J3.7, J3.8
Changed lines of the file:
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@@
 	)
 	(junction
-		(at 123.19 69.85)
+		(at 215.9 72.39)
 		(diameter 0)
 		(color 0 0 0 0)
 	)
 	(junction
-		(at 40.64 95.25)
+		(at 123.19 69.85)
 		(diameter 0)
 		(color 0 0 0 0)
 	)
 	(junction
-		(at 133.35 151.13)
+		(at 40.64 95.25)
 		(diameter 0)
 		(color 0 0 0 0)
 	)
 	(junction
-		(at 151.13 151.13)
+		(at 215.9 80.01)
 		(diameter 0)
 		(color 0 0 0 0)
 	)
 	(junction
-		(at 187.96 74.93)
+		(at 133.35 151.13)
 		(diameter 0)
 		(color 0 0 0 0)
 	)
 	(junction
-		(at 59.69 130.81)
+		(at 151.13 151.13)
 		(diameter 0)
 		(color 0 0 0 0)
 	)
 	(junction
-		(at 133.35 137.16)
+		(at 187.96 74.93)
 		(diameter 0)
 		(color 0 0 0 0)
 	)
 	(junction
-		(at 151.13 137.16)
+		(at 59.69 130.81)
 		(diameter 0)
 		(color 0 0 0 0)
 	)
 	(junction
-		(at 215.9 80.01)
+		(at 133.35 137.16)
 		(diameter 0)
 		(color 0 0 0 0)
 	)
 	(junction
-		(at 215.9 72.39)
+		(at 151.13 137.16)
 		(diameter 0)
 		(color 0 0 0 0)
@@
 	(wire
 		(pts
+			(xy 229.87 52.07) (xy 229.87 55.88)
+		)
+		(stroke
+			(width 0)
+			(type default)
+		)
+	)
+	(wire
+		(pts
 			(xy 29.21 82.55) (xy 53.34 82.55)
 		)
@@
 	(wire
 		(pts
+			(xy 226.06 52.07) (xy 229.87 52.07)
+		)
+		(stroke
+			(width 0)
+			(type default)
+		)
+	)
+	(wire
+		(pts
 			(xy 107.95 74.93) (xy 118.11 74.93)
 		)
@@
 	(wire
 		(pts
+			(xy 226.06 57.15) (xy 226.06 52.07)
+		)
+		(stroke
+			(width 0)
+			(type default)
+		)
+	)
+	(wire
+		(pts
 			(xy 170.18 34.29) (xy 172.72 34.29)
 		)
@@
 	)
 	(symbol
-		(lib_id "Connector:RJ45_LED")
-		(at 226.06 69.85 180)
-		(unit 1)
-		(exclude_from_sim yes)
-		(in_bom yes)
-		(on_board yes)
-		(dnp no)
-		(fields_autoplaced yes)
-		(property "Reference" "J3"
-			(at 226.06 54.61 0)
-			(effects
-				(font
-					(size 1.27 1.27)
-				)
-			)
-		)
-		(property "Value" "RJ45_LED"
-			(at 226.06 57.15 0)
-			(effects
-				(font
-					(size 1.27 1.27)
-				)
-			)
-		)
-		(property "Footprint" ""
-			(at 226.06 70.485 90)
-			(effects
-				(font
-					(size 1.27 1.27)
-				)
-				(hide yes)
-			)
-		)
-		(property "Datasheet" "~"
-			(at 226.06 70.485 90)
-			(effects
-				(font
-					(size 1.27 1.27)
-				)
-				(hide yes)
-			)
-		)
-		(property "Description" "RJ connector, 8P8C (8 positions 8 connected), two LEDs"
-			(at 226.06 69.85 0)
-			(effects
-				(font
-					(size 1.27 1.27)
-				)
-				(hide yes)
-			)
-		)
-		(pin "12"
-		)
-		(pin "11"
-		)
-		(pin "10"
-		)
-		(pin "1"
-		)
-		(pin "3"
-		)
-		(pin "7"
-		)
-		(pin "4"
-		)
-		(pin "5"
-		)
-		(pin "2"
-		)
-		(pin "9"
-		)
-		(pin "8"
-		)
-		(pin "6"
-		)
-		(instances
-			(project "asynthosc"
-				(path "/d73e377a-a016-415f-8824-91cc6e4907b9/dee5e89d-6774-4f8d-b6d8-6a859b9e32e8/354f1097-74a0-4bc1-8721-d2c0e4c9dab3"
-					(reference "J3")
-					(unit 1)
-				)
-			)
-		)
-	)
-	(symbol
 		(lib_id "Device:Crystal")
 		(at 59.69 111.76 0)
@@
 	)
 	(symbol
+		(lib_id "Connector:RJ45_LED_Shielded")
+		(at 226.06 69.85 180)
+		(unit 1)
+		(exclude_from_sim no)
+		(in_bom yes)
+		(on_board yes)
+		(dnp no)
+		(property "Reference" "J3"
+			(at 225.552 84.328 0)
+			(effects
+				(font
+					(size 1.27 1.27)
+				)
+			)
+		)
+		(property "Value" "RJ45_LED_Shielded"
+			(at 226.06 86.36 0)
+			(effects
+				(font
+					(size 1.27 1.27)
+				)
+			)
+		)
+		(property "Footprint" "asynthosc:RJ45_HCTL_HC-RJ45-053-2"
+			(at 226.06 70.485 90)
+			(effects
+				(font
+					(size 1.27 1.27)
+				)
+				(hide yes)
+			)
+		)
+		(property "Datasheet" "~"
+			(at 226.06 70.485 90)
+			(effects
+				(font
+					(size 1.27 1.27)
+				)
+				(hide yes)
+			)
+		)
+		(property "Description" "RJ connector, 8P8C (8 positions 8 connected), two LEDs, Shielded"
+			(at 226.06 69.85 0)
+			(effects
+				(font
+					(size 1.27 1.27)
+				)
+				(hide yes)
+			)
+		)
+		(pin "3"
+		)
+		(pin "4"
+		)
+		(pin "8"
+		)
+		(pin "9"
+		)
+		(pin "6"
+		)
+		(pin "SH"
+		)
+		(pin "7"
+		)
+		(pin "11"
+		)
+		(pin "10"
+		)
+		(pin "2"
+		)
+		(pin "12"
+		)
+		(pin "5"
+		)
+		(pin "1"
+		)
+		(instances
+			(project ""
+				(path "/d73e377a-a016-415f-8824-91cc6e4907b9/dee5e89d-6774-4f8d-b6d8-6a859b9e32e8/354f1097-74a0-4bc1-8721-d2c0e4c9dab3"
+					(reference "J3")
+					(unit 1)
+				)
+			)
+		)
+	)
+	(symbol
 		(lib_id "Device:FerriteBead")
 		(at 91.44 31.75 270)
@@
 			)
 		)
-		(property "Footprint" ""
+		(property "Footprint" "Inductor_SMD:L_0402_1005Metric"
 			(at 91.44 29.972 90)
 			(effects
@@
 					(unit 1)
 				)
+			)
+		)
+	)
+	(symbol
+		(lib_id "power:GND")
+		(at 229.87 55.88 0)
+		(unit 1)
+		(exclude_from_sim no)
+		(in_bom yes)
+		(on_board yes)
+		(dnp no)
+		(fields_autoplaced yes)
+		(property "Reference" "#PWR0136"
+			(at 229.87 62.23 0)
+			(effects
+				(font
+					(size 1.27 1.27)
+				)
+				(hide yes)
+			)
+		)
+		(property "Value" "GND"
+			(at 229.87 60.96 0)
+			(effects
+				(font
+					(size 1.27 1.27)
+				)
+				(hide yes)
+			)
+		)
+		(property "Footprint" ""
+			(at 229.87 55.88 0)
+			(effects
+				(font
+					(size 1.27 1.27)
+				)
+				(hide yes)
+			)
+		)
+		(property "Datasheet" ""
+			(at 229.87 55.88 0)
+			(effects
+				(font
+					(size 1.27 1.27)
+				)
+				(hide yes)
+			)
+		)
+		(property "Description" "Power symbol creates a global label with name \"GND\" , ground"
+			(at 229.87 55.88 0)
+			(effects
+				(font
+					(size 1.27 1.27)
+				)
+				(hide yes)
+			)
+		)
+		(pin "1"
+		)
+		(instances
+			(project "asynthosc"
+				(path "/d73e377a-a016-415f-8824-91cc6e4907b9/dee5e89d-6774-4f8d-b6d8-6a859b9e32e8/354f1097-74a0-4bc1-8721-d2c0e4c9dab3"
+					(reference "#PWR0136")
+					(unit 1)
+				)

Commit message: sch: change stm32 for smaller one, create smaller jumper footprint
Parts:
- C31, C32, C33, C34, C35, C36, C37, C39, C40, C41, C42: RefNum (none) -> _generic_
- FB3: Manufacturer (none) -> Murata; RefNum (none) -> BLM15PX330SN1D
- J3: Manufacturer (none) -> HCTL; RefNum (none) -> HC-RJ45-053-2
- JP4: footprint Jumper:SolderJumper-2_P1.3mm_Bridged2Bar_Pad1.0x1.5mm -> asynthosc:SolderJumper_0402_1005Metric_Bridged
- TR1: RefNum (none) -> PT61017PEL
- U5: Manufacturer (none) -> Microchip; RefNum (none) -> LAN8742A
- U6: Manufacturer (none) -> ST; RefNum (none) -> USBLC6-2P6
