File: kicad/asynthosc/soc.kicad_sch (KiCad schematic)
At the start: 46 parts, among them J3 Conn_ARM_SWD_TagConnect_TC203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, J4 Conn_02x07_Odd_Even, J5 Conn_02x04_Odd_Even, SW1 SW_Push, U6 STM32F723VETx, U7 W25Q32JVSS, Y1 8MHz, 8pF

Commit message: pcb: routing
Connections:
- net DISP_10V_EN: now also U6.56 (PB14)
- net DISP_DC: now also U6.62 (PD15)
- net DISP_nCS: now also U6.64 (PC7)
- net DISP_nRST: now also U6.63 (PC6)
- net TIM1_CH4: now reaches U6.44 (PE14)
- net DISP_12V_EN: now reaches U6.57 (PB15)
- net LED_BTN_2: now reaches U6.58 (PD11)
- net BTN_2: now reaches U6.59 (PD12)
- net ROT_A: now reaches U6.65 (PC8)
- net ROT_B: now reaches U6.66 (PC9)
- net BTN_1: now reaches U6.83 (PD2)
- net LED_BTN_1: now reaches U6.84 (PD3)
Changed lines of the file:
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@@
+	(wire
+		(pts
+			(xy 152.4 153.67) (xy 158.75 153.67)
+		)
+		(stroke
+			(width 0)
+			(type default)
+		)
+	)
 	(wire
 		(pts
@@
 	(wire
 		(pts
+			(xy 83.82 148.59) (xy 101.6 148.59)
+		)
+		(stroke
+			(width 0)
+			(type default)
+		)
+	)
+	(wire
+		(pts
 			(xy 49.53 27.94) (xy 55.88 27.94)
 		)
@@
 	(wire
 		(pts
+			(xy 92.71 118.11) (xy 101.6 118.11)
+		)
+		(stroke
+			(width 0)
+			(type default)
+		)
+	)
+	(wire
+		(pts
 			(xy 96.52 80.01) (xy 96.52 77.47)
 		)
@@
 	(wire
 		(pts
+			(xy 152.4 156.21) (xy 158.75 156.21)
+		)
+		(stroke
+			(width 0)
+			(type default)
+		)
+	)
+	(wire
+		(pts
+			(xy 152.4 158.75) (xy 158.75 158.75)
+		)
+		(stroke
+			(width 0)
+			(type default)
+		)
+	)
+	(wire
+		(pts
 			(xy 218.44 114.3) (xy 233.68 114.3)
 		)
@@
 	(wire
 		(pts
+			(xy 83.82 146.05) (xy 101.6 146.05)
+		)
+		(stroke
+			(width 0)
+			(type default)
+		)
+	)
+	(wire
+		(pts
 			(xy 101.6 161.29) (xy 88.9 161.29)
 		)
@@
 	(wire
 		(pts
+			(xy 83.82 156.21) (xy 101.6 156.21)
+		)
+		(stroke
+			(width 0)
+			(type default)
+		)
+	)
+	(wire
+		(pts
+			(xy 152.4 130.81) (xy 158.75 130.81)
+		)
+		(stroke
+			(width 0)
+			(type default)
+		)
+	)
+	(wire
+		(pts
 			(xy 49.53 52.07) (xy 52.07 52.07)
 		)
@@
 	(wire
 		(pts
+			(xy 152.4 161.29) (xy 158.75 161.29)
+		)
+		(stroke
+			(width 0)
+			(type default)
+		)
+	)
+	(wire
+		(pts
 			(xy 334.01 78.74) (xy 370.84 78.74)
 		)
@@
 	(wire
 		(pts
+			(xy 83.82 130.81) (xy 101.6 130.81)
+		)
+		(stroke
+			(width 0)
+			(type default)
+		)
+	)
+	(wire
+		(pts
 			(xy 300.99 90.17) (xy 303.53 90.17)
 		)
@@
 	(wire
 		(pts
+			(xy 83.82 133.35) (xy 101.6 133.35)
+		)
+		(stroke
+			(width 0)
+			(type default)
+		)
+	)
+	(wire
+		(pts
 			(xy 218.44 124.46) (xy 233.68 124.46)
 		)
@@
 		(pts
 			(xy 163.83 105.41) (xy 162.56 105.41)
+		)
+		(stroke
+			(width 0)
+			(type default)
+		)
+	)
+	(wire
+		(pts
+			(xy 152.4 133.35) (xy 158.75 133.35)
 		)
 		(stroke
@@
 		)
 	)
+	(hierarchical_label "LED_BTN_1"
+		(shape output)
+		(at 83.82 133.35 180)
+		(fields_autoplaced yes)
+		(effects
+			(font
+				(size 1.27 1.27)
+			)
+			(justify right)
+		)
+	)
 	(hierarchical_label "ADC1_IN0"
 		(shape input)
@@
 		)
 	)
+	(hierarchical_label "BTN_1"
+		(shape input)
+		(at 83.82 130.81 180)
+		(fields_autoplaced yes)
+		(effects
+			(font
+				(size 1.27 1.27)
+			)
+			(justify right)
+		)
+	)
 	(hierarchical_label "ADC1_IN3"
 		(shape input)
@@
 	(hierarchical_label "DISP_10V_EN"
 		(shape output)
-		(at 39.37 119.38 180)
+		(at 54.61 139.7 180)
 		(fields_autoplaced yes)
 		(effects
@@
 			)
 			(justify right)
+		)
+	)
+	(hierarchical_label "ROT_A"
+		(shape input)
+		(at 158.75 158.75 0)
+		(fields_autoplaced yes)
+		(effects
+			(font
+				(size 1.27 1.27)
+			)
+			(justify left)
 		)
 	)
 	(hierarchical_label "DISP_nCS"
 		(shape output)
-		(at 39.37 128.27 180)
-		(fields_autoplaced yes)
-		(effects
-			(font
-				(size 1.27 1.27)
-			)
-			(justify right)
+		(at 158.75 156.21 0)
+		(fields_autoplaced yes)
+		(effects
+			(font
+				(size 1.27 1.27)
+			)
+			(justify left)
 		)
 	)
@@
 		)
 	)
+	(hierarchical_label "BTN_2"
+		(shape input)
+		(at 83.82 148.59 180)
+		(fields_autoplaced yes)
+		(effects
+			(font
+				(size 1.27 1.27)
+			)
+			(justify right)
+		)
+	)
 	(hierarchical_label "UART4_TX"
 		(shape output)
@@
 	(hierarchical_label "DISP_DC"
 		(shape output)
-		(at 39.37 125.73 180)
+		(at 83.82 156.21 180)
+		(fields_autoplaced yes)
+		(effects
+			(font
+				(size 1.27 1.27)
+			)
+			(justify right)
+		)
+	)
+	(hierarchical_label "TIM1_CH4"
+		(shape input)
+		(at 92.71 118.11 180)
 		(fields_autoplaced yes)
 		(effects
@@
 		)
 	)
+	(hierarchical_label "LED_BTN_2"
+		(shape output)
+		(at 83.82 146.05 180)
+		(fields_autoplaced yes)
+		(effects
+			(font
+				(size 1.27 1.27)
+			)
+			(justify right)
+		)
+	)
+	(hierarchical_label "ROT_B"
+		(shape input)
+		(at 158.75 161.29 0)
+		(fields_autoplaced yes)
+		(effects
+			(font
+				(size 1.27 1.27)
+			)
+			(justify left)
+		)
+	)
 	(hierarchical_label "ADC1_IN5"
 		(shape input)
@@
 	(hierarchical_label "DISP_nRST"
 		(shape output)
-		(at 39.37 123.19 180)
-		(fields_autoplaced yes)
-		(effects
-			(font
-				(size 1.27 1.27)
-			)
-			(justify right)
+		(at 158.75 153.67 0)
+		(fields_autoplaced yes)
+		(effects
+			(font
+				(size 1.27 1.27)
+			)
+			(justify left)
+		)
+	)
+	(hierarchical_label "DISP_10V_EN"
+		(shape output)
+		(at 158.75 130.81 0)
+		(fields_autoplaced yes)
+		(effects
+			(font
+				(size 1.27 1.27)
+			)
+			(justify left)
 		)
 	)
@@
 		)
 	)
+	(hierarchical_label "DISP_12V_EN"
+		(shape output)
+		(at 158.75 133.35 0)
+		(fields_autoplaced yes)
+		(effects
+			(font
+				(size 1.27 1.27)
+			)
+			(justify left)
+		)
+	)
