File: kicad/asynthosc/asynthosc.kicad_sch (KiCad schematic)
At the start: 34 parts

Commit message: bom: update for better bom
Parts:
- FID1, FID2, FID3, FID4, H4, H5, H6, H7, MB1, MB2, MB3, MB4, MB5, MB6, MB7, MB8: RefNum (none) -> _na_
Changed lines of the file:
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@@
+			)
+		)
+		(property "RefNum" "_na_"
+			(at 50.8 39.37 0)
+			(effects
+				(font
+					(size 1.27 1.27)
+				)
+				(hide yes)
 			)
 		)
@@
 			)
 		)
+		(property "RefNum" "_na_"
+			(at 31.75 33.02 0)
+			(effects
+				(font
+					(size 1.27 1.27)
+				)
+				(hide yes)
+			)
+		)
 		(instances
 			(project "asynthosc"
@@
 		)
 		(property "Description" "Mouse Bytes"
+			(at 76.2 29.21 0)
+			(effects
+				(font
+					(size 1.27 1.27)
+				)
+				(hide yes)
+			)
+		)
+		(property "RefNum" "_na_"
 			(at 76.2 29.21 0)
 			(effects
@@
 			)
 		)
+		(property "RefNum" "_na_"
+			(at 31.75 20.32 0)
+			(effects
+				(font
+					(size 1.27 1.27)
+				)
+				(hide yes)
+			)
+		)
 		(instances
 			(project ""
@@
 			)
 		)
+		(property "RefNum" "_na_"
+			(at 50.8 20.32 0)
+			(effects
+				(font
+					(size 1.27 1.27)
+				)
+				(hide yes)
+			)
+		)
 		(instances
 			(project ""
@@
 			)
 		)
+		(property "RefNum" "_na_"
+			(at 76.2 34.29 0)
+			(effects
+				(font
+					(size 1.27 1.27)
+				)
+				(hide yes)
+			)
+		)
 		(instances
 			(project "asynthosc"
@@
 			)
 		)
+		(property "RefNum" "_na_"
+			(at 31.75 26.67 0)
+			(effects
+				(font
+					(size 1.27 1.27)
+				)
+				(hide yes)
+			)
+		)
 		(instances
 			(project "asynthosc"
@@
 			)
 		)
+		(property "RefNum" "_na_"
+			(at 31.75 39.37 0)
+			(effects
+				(font
+					(size 1.27 1.27)
+				)
+				(hide yes)
+			)
+		)
 		(instances
 			(project "asynthosc"
@@
 			)
 		)
+		(property "RefNum" "_na_"
+			(at 76.2 21.59 0)
+			(effects
+				(font
+					(size 1.27 1.27)
+				)
+				(hide yes)
+			)
+		)
 		(instances
 			(project ""
@@
 		)
 		(property "Description" "Mouse Bytes"
+			(at 76.2 39.37 0)
+			(effects
+				(font
+					(size 1.27 1.27)
+				)
+				(hide yes)
+			)
+		)
+		(property "RefNum" "_na_"
 			(at 76.2 39.37 0)
 			(effects
@@
 			)
 		)
+		(property "RefNum" "_na_"
+			(at 50.8 33.02 0)
+			(effects
+				(font
+					(size 1.27 1.27)
+				)
+				(hide yes)
+			)
+		)
 		(instances
 			(project "asynthosc"
@@
 			)
 		)
+		(property "RefNum" "_na_"
+			(at 76.2 36.83 0)
+			(effects
+				(font
+					(size 1.27 1.27)
+				)
+				(hide yes)
+			)
+		)
 		(instances
 			(project "asynthosc"
@@
 			)
 		)
+		(property "RefNum" "_na_"
+			(at 76.2 31.75 0)
+			(effects
+				(font
+					(size 1.27 1.27)
+				)
+				(hide yes)
+			)
+		)
 		(instances
 			(project "asynthosc"
@@
 			)
 		)
+		(property "RefNum" "_na_"
+			(at 50.8 26.67 0)
+			(effects
+				(font
+					(size 1.27 1.27)
+				)
+				(hide yes)
+			)
+		)
 		(instances
 			(project "asynthosc"
@@
 		)
 		(property "Description" "Mouse Bytes"
+			(at 76.2 26.67 0)
+			(effects
+				(font
+					(size 1.27 1.27)
+				)
+				(hide yes)
+			)
+		)
+		(property "RefNum" "_na_"
 			(at 76.2 26.67 0)
 			(effects
@@
 			(at 76.2 24.13 0)
 			(effects
+				(font
+					(size 1.27 1.27)
+				)
+				(hide yes)
+			)
+		)
+		(property "RefNum" "_na_"
+			(at 76.2 24.13 0)
+			(effects
